Commit message: Deleted original launch files (have been moved to /launch)

File: umi_rtx_100.urdf (robot description, URDF)
Before this commit: robot HSRDP, 7 links, 6 joints
Links:
- removed link wrist_gearbox_pitch
- removed link wrist_gearbox_roll
- added link gripper; visual mesh filename=package://moveit_hsrdp/meshes/l_finger.dae
- added link virtual_link
- added link wrist; visual box size=0.10 0.10 0.05
Joints:
- removed joint wrist_pitch
- removed joint wrist_roll
- added joint gripper_pitch: type revolute, parent virtual_link, child wrist, origin xyz=0 0 0, axis 0 -1 0, limit lower=-1.71 upper=0.07 effort=1 velocity=1
- added joint gripper_roll: type revolute, parent wrist_to_gripper, child virtual_link, origin xyz=0 0 0, axis -1 0 0, limit lower=-3.16 upper=2.3 effort=1 velocity=1
- added joint wrist_gripper_connection: type fixed, parent wrist, child gripper, origin xyz=0 0 0

Commit message: Restructured the urdf. Removed the two links to deal with gripper movement. virtual_joint is used.

File: umi_rtx_100.urdf (robot description, URDF)
Before this commit: robot HSRDP, 8 links, 7 joints
Links:
- removed link wrist
- removed link wrist_to_gripper
- added link wrist_gripper_connection_to_gripper; visual box size=0.075 0.10 0.05
- added link wrist_to_wrist_gripper_connection; visual box size=0.10 0.10 0.05
- link gripper: geometry visual box size=0.10 0.10 0.02
Joints:
- removed joint gripper_pitch
- removed joint gripper_roll
- removed joint wrist_yaw
- added joint wrist: type revolute, parent elbow_to_wrist, child wrist_to_wrist_gripper_connection, origin xyz=0.252 0 -0.05, axis 0 0 1, limit lower=-1.92 upper=1.92 effort=1 velocity=1
- added joint wrist_gripper_connection_pitch: type revolute, parent virtual_link, child wrist_gripper_connection_to_gripper, origin xyz=0 0 0, axis 0 -1 0, limit lower=-1.71 upper=0.07 effort=1 velocity=1
- added joint wrist_gripper_connection_roll: type revolute, parent wrist_to_wrist_gripper_connection, child virtual_link, origin xyz=0 0 0, axis -1 0 0, limit lower=-3.16 upper=2.3 effort=1 velocity=1
- joint wrist_gripper_connection: parent wrist -> wrist_gripper_connection_to_gripper

Commit message: Got to a basic working state displaying real arm data.

File: umi_rtx_100.urdf (robot description, URDF)
Before this commit: robot HSRDP, 8 links, 7 joints
Links:
- removed link gripper
- removed link shoulder
- added link gripper_base; visual box size=0.11 0.095 0.018
- added link shoulder_link; visual box size=0.278 0.132 0.091
- link wrist_gripper_connection_to_gripper: geometry visual box size=0.10 0.10 0.05
- link wrist_to_wrist_gripper_connection: geometry visual box size=0.075 0.10 0.05
Joints:
- removed joint shoulder
- added joint shoulder_joint: type revolute, parent shoulder_link, child shoulder_to_elbow, origin xyz=-0.01 0 -0.09, axis 0 0 1, limit lower=-1.57 upper=1.57 effort=1 velocity=1
- joint shoulder_updown: child shoulder -> shoulder_link
- joint wrist_gripper_connection: child gripper -> gripper_base
