Commit message: metapackage conversion

File: hsrdp_bridge/umi_rtx_100.urdf (robot description, URDF)
Before this commit: robot HSRDP, 7 links, 6 joints
Links:
- removed link shoulder
- removed link wrist_gearbox_pitch
- removed link wrist_gearbox_roll
- removed link wrist_to_gripper
- added link gripper_base; visual box size=0.11 0.095 0.018
- added link shoulder_link; visual box size=0.278 0.132 0.091
- added link virtual_link
- added link wrist_gripper_connection_to_gripper; visual box size=0.10 0.10 0.05
- added link wrist_to_wrist_gripper_connection; visual box size=0.075 0.10 0.05
Joints:
- removed joint shoulder
- removed joint wrist_pitch
- removed joint wrist_roll
- removed joint wrist_yaw
- added joint shoulder_joint: type revolute, parent shoulder_link, child shoulder_to_elbow, origin xyz=-0.01 0 -0.09, axis 0 0 1, limit lower=-1.57 upper=1.57 effort=1 velocity=1
- added joint wrist: type revolute, parent elbow_to_wrist, child wrist_to_wrist_gripper_connection, origin xyz=0.252 0 -0.05, axis 0 0 1, limit lower=-1.92 upper=1.92 effort=1 velocity=1
- added joint wrist_gripper_connection: type fixed, parent wrist_gripper_connection_to_gripper, child gripper_base, origin xyz=0 0 0
- added joint wrist_gripper_connection_pitch: type revolute, parent virtual_link, child wrist_gripper_connection_to_gripper, origin xyz=0 0 0, axis 0 -1 0, limit lower=-1.71 upper=0.07 effort=1 velocity=1
- added joint wrist_gripper_connection_roll: type revolute, parent wrist_to_wrist_gripper_connection, child virtual_link, origin xyz=0 0 0, axis -1 0 0, limit lower=-3.16 upper=2.3 effort=1 velocity=1
- joint shoulder_updown: child shoulder -> shoulder_link

Commit message: Started changes to urdf and srdf to add placeholder gripper model.

File: hsrdp_bridge/umi_rtx_100.urdf (robot description, URDF)
Before this commit: robot HSRDP, 8 links, 7 joints
Links:
- added link left_finger; visual box size=0.07 0.015 0.025
- added link right_finger; visual box size=0.07 0.015 0.025
- link gripper_base: geometry visual box size=0.077 0.15 0.078
Joints:
- added joint gripper_left: type prismatic, parent gripper_base, child left_finger, origin xyz=0 0 0, axis 0 -1 0, limit lower=-1.71 upper=0.07 effort=1 velocity=1
- added joint gripper_right: type prismatic, parent gripper_base, child right_finger, origin xyz=0 0 0, axis 0 -1 0, limit lower=-1.71 upper=0.07 effort=1 velocity=1

Commit message: Commited changes when AlexR rushed off :P

File: hsrdp_bridge/umi_rtx_100.urdf (robot description, URDF)
Before this commit: robot HSRDP, 10 links, 9 joints
Joints:
- joint gripper_left: axis 0 -1 0 -> 0 0 -1; limit lower=-1.71 upper=0.07 effort=1 velocity=1 -> lower=-0.15 upper=0.06 effort=1 velocity=1; origin xyz=0 0 0 -> xyz=0 0 0 rpy=0 -0.1 0; type prismatic -> revolute
- joint gripper_right: axis 0 -1 0 -> 0 0 -1; limit lower=-1.71 upper=0.07 effort=1 velocity=1 -> lower=-0.15 upper=0.06 effort=1 velocity=1; mimic (none) -> joint=gripper_left multiplier=-1; origin xyz=0 0 0 -> xyz=0 0 0 rpy=0 -0.1 0; type prismatic -> revolute

Commit message: Used move_group interface to plan/execute end-effector through setPoseTarget. Gripper not moving yet through setJointValue but other joints are fine.

File: hsrdp_bridge/umi_rtx_100.urdf (robot description, URDF)
Before this commit: robot HSRDP, 10 links, 9 joints
Joints:
- joint gripper_left: origin xyz=0 0 0 rpy=0 -0.1 0 -> xyz=0 0 0 rpy=0 0 0
- joint gripper_right: origin xyz=0 0 0 rpy=0 -0.1 0 -> xyz=0 0 0 rpy=0 0 0

Commit message: Gripper can be set from move group interface

File: hsrdp_bridge/umi_rtx_100.urdf (robot description, URDF)
Before this commit: robot HSRDP, 10 links, 9 joints
Joints:
- joint gripper_right: limit lower=-0.15 upper=0.06 effort=1 velocity=1 -> lower=-0.06 upper=0.15 effort=1 velocity=1

Commit message: Traces out 3x3 horizontal square then closes gripper. (Only tested in simulation)

File: hsrdp_bridge/umi_rtx_100.urdf (robot description, URDF)
Before this commit: robot HSRDP, 10 links, 9 joints
Joints:
- joint gripper_left: limit lower=-0.15 upper=0.06 effort=1 velocity=1 -> lower=-0.3 upper=0.06 effort=1 velocity=1; origin xyz=0 0 0 rpy=0 0 0 -> xyz=0.12 0 0 rpy=0 0 0
- joint gripper_right: limit lower=-0.06 upper=0.15 effort=1 velocity=1 -> lower=-0.06 upper=0.3 effort=1 velocity=1; origin xyz=0 0 0 rpy=0 0 0 -> xyz=0.12 0 0 rpy=0 0 0

Commit message: Many changes moving towards getting the gripper working with the movegroup.

File: hsrdp_bridge/umi_rtx_100.urdf (robot description, URDF)
Before this commit: robot HSRDP, 10 links, 9 joints
Joints:
- joint gripper_left: axis 0 0 -1 -> 0 1 0; limit lower=-0.3 upper=0.06 effort=1 velocity=1 -> lower=0 upper=0.05 effort=1 velocity=1; type revolute -> prismatic
- joint gripper_right: axis 0 0 -1 -> 0 1 0 ; limit lower=-0.06 upper=0.3 effort=1 velocity=1 -> lower=-0.05 upper=0 effort=1 velocity=1; type revolute -> prismatic

Commit message: Gripper movement happens first. Slight change (by eye) to be closer to actual z-axis positions.

File: hsrdp_bridge/umi_rtx_100.urdf (robot description, URDF)
Before this commit: robot HSRDP, 10 links, 9 joints
Joints:
- joint shoulder_updown: origin xyz=0.0445 0 0.134 -> xyz=0.0445 0 -0.3
